File: Circuitos/Segundero con 555 [Kicad]/Segundero 555.kicad_sch (KiCad schematic)
At the start: 20 parts, among them J1 Screw_Terminal_01x02, U1 7447, U2 7490, U3 NE555P

Commit message: .
Parts:
- C2: footprint Capacitor_THT:CP_Radial_D4.0mm_P2.00mm -> Capacitor_THT:CP_Radial_D8.0mm_P3.80mm
- J1: value Screw_Terminal_01x02 -> 5V in; footprint (none) -> TerminalBlock_Phoenix:TerminalBlock_Phoenix_MKDS-1,5-2_1x02_P5.00mm_Horizontal
Connections:
- net +5V: no longer R4.1, R5.1, R6.1, R7.1, U1.1 (B), U1.2 (C), U1.6 (D), U1.7 (A), U2.1 (~{CKB}), U2.11 (Q3), U2.12 (Q0), U2.8 (Q2), U2.9 (Q1)
- new net: R6.1, U1.1 (B), U2.9 (Q1)
- new net: R5.1, U1.2 (C), U2.8 (Q2)
- new net: R4.1, U1.6 (D), U2.11 (Q3)
- new net: R7.1, U1.7 (A), U2.1 (~{CKB}), U2.12 (Q0)
Changed lines of the file:
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@@
   (junction (at 95.25 44.45) (diameter 0) (color 0 0 0 0)
   )
-  (junction (at 180.34 53.34) (diameter 0) (color 0 0 0 0)
-  )
   (junction (at 73.66 58.42) (diameter 0) (color 0 0 0 0)
   )
@@
   (junction (at 147.32 62.23) (diameter 0) (color 0 0 0 0)
   )
-  (junction (at 180.34 48.26) (diameter 0) (color 0 0 0 0)
-  )
   (junction (at 26.67 58.42) (diameter 0) (color 0 0 0 0)
   )
@@
   (junction (at 26.67 43.18) (diameter 0) (color 0 0 0 0)
   )
-  (junction (at 180.34 38.1) (diameter 0) (color 0 0 0 0)
-  )
   (junction (at 152.4 67.31) (diameter 0) (color 0 0 0 0)
   )
   (junction (at 146.05 72.39) (diameter 0) (color 0 0 0 0)
   )
-  (junction (at 180.34 43.18) (diameter 0) (color 0 0 0 0)
-  )
   (junction (at 137.16 62.23) (diameter 0) (color 0 0 0 0)
   )
   (junction (at 26.67 77.47) (diameter 0) (color 0 0 0 0)
   )
+  (junction (at 180.34 60.96) (diameter 0) (color 0 0 0 0)
+  )
   (junction (at 95.25 49.53) (diameter 0) (color 0 0 0 0)
   )
   (junction (at 180.34 66.04) (diameter 0) (color 0 0 0 0)
   )
-  (junction (at 180.34 60.96) (diameter 0) (color 0 0 0 0)
-  )
   (junction (at 95.25 46.99) (diameter 0) (color 0 0 0 0)
   )
@@
     (stroke (width 0) (type default))
   )
-  (wire (pts (xy 180.34 38.1) (xy 180.34 43.18))
-    (stroke (width 0) (type default))
-  )
   (wire (pts (xy 95.25 46.99) (xy 95.25 44.45))
     (stroke (width 0) (type default))
@@
     (stroke (width 0) (type default))
   )
-  (wire (pts (xy 180.34 53.34) (xy 180.34 60.96))
-    (stroke (width 0) (type default))
-  )
   (wire (pts (xy 224.79 40.64) (xy 224.79 48.26))
     (stroke (width 0) (type default))
@@
     (stroke (width 0) (type default))
   )
-  (wire (pts (xy 180.34 43.18) (xy 180.34 48.26))
-    (stroke (width 0) (type default))
-  )
   (wire (pts (xy 180.34 71.12) (xy 180.34 66.04))
     (stroke (width 0) (type default))
@@
     (stroke (width 0) (type default))
   )
-  (wire (pts (xy 180.34 48.26) (xy 180.34 53.34))
-    (stroke (width 0) (type default))
-  )
   (wire (pts (xy 95.25 49.53) (xy 95.25 46.99))
     (stroke (width 0) (type default))
@@
     (stroke (width 0) (type default))
   )
-  (wire (pts (xy 180.34 25.4) (xy 180.34 38.1))
-    (stroke (width 0) (type default))
-  )
   (wire (pts (xy 40.64 68.58) (xy 33.02 68.58))
     (stroke (width 0) (type default))
@@
     )
   )
-  (symbol (lib_id "power:+5V") (at 180.34 25.4 0) (unit 1)
+  (symbol (lib_id "power:+5V") (at 180.34 60.96 0) (unit 1)
     (in_bom yes) (on_board yes) (dnp no)
-    (property "Reference" "#PWR05" (at 180.34 29.21 0)
+    (property "Reference" "#PWR05" (at 180.34 64.77 0)
       (effects (font (size 1.27 1.27)) hide)
     )
-    (property "Value" "+5V" (at 180.34 21.59 0)
+    (property "Value" "+5V" (at 180.34 57.15 0)
       (effects (font (size 1.27 1.27)))
     )
-    (property "Footprint" "" (at 180.34 25.4 0)
+    (property "Footprint" "" (at 180.34 60.96 0)
       (effects (font (size 1.27 1.27)) hide)
     )
-    (property "Datasheet" "" (at 180.34 25.4 0)
+    (property "Datasheet" "" (at 180.34 60.96 0)
       (effects (font (size 1.27 1.27)) hide)
     )
@@
       (effects (font (size 1.27 1.27)) (justify left))
     )
-    (property "Footprint" "Capacitor_THT:CP_Radial_D4.0mm_P2.00mm" (at 27.6352 91.44 0)
+    (property "Footprint" "Capacitor_THT:CP_Radial_D8.0mm_P3.80mm" (at 27.6352 91.44 0)
       (effects (font (size 1.27 1.27)) hide)
     )
@@
   )
   (symbol (lib_id "Connector:Screw_Terminal_01x02") (at 26.67 118.11 180) (unit 1)
-    (in_bom yes) (on_board yes) (dnp no) (fields_autoplaced)
+    (in_bom yes) (on_board yes) (dnp no)
     (property "Reference" "J1" (at 26.67 111.76 0)
       (effects (font (size 1.27 1.27)))
     )
-    (property "Value" "Screw_Terminal_01x02" (at 26.67 111.76 0)
-      (effects (font (size 1.27 1.27)) hide)
+    (property "Value" "5V in" (at 22.86 116.84 90)
+      (effects (font (size 1.27 1.27)))
     )
-    (property "Footprint" "" (at 26.67 118.11 0)
+    (property "Footprint" "TerminalBlock_Phoenix:TerminalBlock_Phoenix_MKDS-1,5-2_1x02_P5.00mm_Horizontal" (at 26.67 118.11 0)
       (effects (font (size 1.27 1.27)) hide)
     )
