File: Circuitos/Segundero con 555 [Kicad]/Segundero 555.kicad_pcb (KiCad board)
At the start: 2 copper layers, 80 x 50 mm, 24 parts, among them J1 5V in, U1 7447, U2 7490, U3 NE555P

Commit message: .
Other:
- board text added: "+"
- board text added: "-"
- board text added: "5V"
- board text added: "Bit 0"
- board text added: "Bit 1"
- board text added: "Bit 2"
- board text added: "Bit 3"
Changed lines of the file:
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@@
         (effects (font (size 1 1) (thickness 0.15)))
     )
-    (fp_text value "LTS-6960HR" (at 7.62 12.58 90) (layer "F.Fab")
+    (fp_text value "LTS-6960HR" (at 7.62 12.58 90) (layer "F.SilkS")
         (effects (font (size 1 1) (thickness 0.15)))
     )
@@
         (effects (font (size 1 1) (thickness 0.15)))
     )
-    (fp_text value "7490" (at 3.81 17.57) (layer "F.Fab")
+    (fp_text value "7490" (at 3.81 17.57) (layer "F.SilkS")
         (effects (font (size 1 1) (thickness 0.15)))
     )
@@
     (property "ki_keywords" "LED diode")
     (attr through_hole)
-    (fp_text reference "D1" (at 1.27 -3.96) (layer "F.SilkS")
+    (fp_text reference "D1" (at 4.54 3) (layer "F.SilkS")
         (effects (font (size 1 1) (thickness 0.15)))
     )
@@
         (effects (font (size 1 1) (thickness 0.15)))
     )
-    (fp_text value "7447" (at 3.81 20.11) (layer "F.Fab")
+    (fp_text value "7447" (at 3.81 20.11) (layer "F.SilkS")
         (effects (font (size 1 1) (thickness 0.15)))
     )
@@
         (effects (font (size 1 1) (thickness 0.15)))
     )
-    (fp_text value "NE555P" (at 3.81 -2.2) (layer "F.Fab")
+    (fp_text value "NE555P" (at 3.81 -2.2) (layer "F.SilkS")
         (effects (font (size 1 1) (thickness 0.15)))
     )
@@
   (gr_line (start 160 110) (end 160 60)
     (stroke (width 0.05) (type default)) (layer "Edge.Cuts"))
+  (gr_text "Bit 0" (at 125.5 108.5) (layer "F.SilkS")
+    (effects (font (size 1 1) (thickness 0.1)) (justify left bottom))
+  )
   (gr_text "Segundero con 555 v1.0\nAlejandro Alonso Puig (2024)" (at 158 97 90) (layer "F.SilkS")
     (effects (font (size 1.2 1.2) (thickness 0.1)) (justify left bottom))
   )
+  (gr_text "-" (at 82.5 95.5 90) (layer "F.SilkS")
+    (effects (font (size 1 1) (thickness 0.1)) (justify left bottom))
+  )
+  (gr_text "Bit 1" (at 118 108.5) (layer "F.SilkS")
+    (effects (font (size 1 1) (thickness 0.1)) (justify left bottom))
+  )
+  (gr_text "+" (at 81 102) (layer "F.SilkS")
+    (effects (font (size 1.5 1.5) (thickness 0.1)) (justify left bottom))
+  )
+  (gr_text "5V" (at 82.5 99 90) (layer "F.SilkS")
+    (effects (font (size 1 1) (thickness 0.1)) (justify left bottom))
+  )
+  (gr_text "Bit 3" (at 103 108.5) (layer "F.SilkS")
+    (effects (font (size 1 1) (thickness 0.1)) (justify left bottom))
+  )
+  (gr_text "Bit 2" (at 110.5 108.5) (layer "F.SilkS")
+    (effects (font (size 1 1) (thickness 0.1)) (justify left bottom))
+  )
   (segment (start 142 98) (end 155 98) (width 0.6) (layer "F.Cu") (net 1))
