File: Circuitos/NE555 frecuencia y pwm [Kicad]/NE555 frecuencia y pwm [Kicad].kicad_sch (KiCad schematic)
At the start: 14 parts, among them J1 Power, J2 Motor, Q1 IRLZ24, U1 NE555P

Commit message: .
Parts:
- renumbered RV1(Frecuencia) to RV1(Frecuencia)1, RV2(Duty) to RV2(Duty)1
Changed lines of the file:
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@@
     (comment 1 "Por: Alejandro Alonso Puig")
   )
+  (junction (at 128.27 71.12) (diameter 0) (color 0 0 0 0)
+  )
+  (junction (at 128.27 113.03) (diameter 0) (color 0 0 0 0)
+  )
   (junction (at 167.64 100.33) (diameter 0) (color 0 0 0 0)
   )
@@
     (stroke (width 0) (type default))
   )
-  (wire (pts (xy 128.27 102.87) (xy 128.27 115.57))
+  (wire (pts (xy 128.27 102.87) (xy 128.27 113.03))
     (stroke (width 0) (type default))
   )
@@
     (stroke (width 0) (type default))
   )
+  (wire (pts (xy 128.27 71.12) (xy 128.27 76.2))
+    (stroke (width 0) (type default))
+  )
+  (wire (pts (xy 128.27 76.2) (xy 139.7 76.2))
+    (stroke (width 0) (type default))
+  )
   (wire (pts (xy 147.32 76.2) (xy 167.64 76.2))
     (stroke (width 0) (type default))
@@
     (stroke (width 0) (type default))
   )
-  (wire (pts (xy 128.27 67.31) (xy 128.27 76.2))
+  (wire (pts (xy 128.27 67.31) (xy 128.27 71.12))
     (stroke (width 0) (type default))
   )
@@
     (stroke (width 0) (type default))
   )
+  (wire (pts (xy 104.14 97.79) (xy 104.14 76.2))
+    (stroke (width 0) (type default))
+  )
+  (wire (pts (xy 162.56 100.33) (xy 167.64 100.33))
+    (stroke (width 0) (type default))
+  )
+  (wire (pts (xy 236.22 83.82) (xy 236.22 81.28))
+    (stroke (width 0) (type default))
+  )
+  (wire (pts (xy 104.14 76.2) (xy 128.27 76.2))
+    (stroke (width 0) (type default))
+  )
+  (wire (pts (xy 140.97 97.79) (xy 143.51 97.79))
+    (stroke (width 0) (type default))
+  )
+  (wire (pts (xy 179.07 110.49) (xy 179.07 113.03))
+    (stroke (width 0) (type default))
+  )
+  (wire (pts (xy 147.32 87.63) (xy 140.97 87.63))
+    (stroke (width 0) (type default))
+  )
+  (wire (pts (xy 179.07 113.03) (xy 179.07 120.65))
+    (stroke (width 0) (type default))
+  )
+  (wire (pts (xy 167.64 100.33) (xy 179.07 100.33))
+    (stroke (width 0) (type default))
+  )
+  (wire (pts (xy 228.6 88.9) (xy 228.6 95.25))
+    (stroke (width 0) (type default))
+  )
+  (wire (pts (xy 228.6 118.11) (xy 228.6 105.41))
+    (stroke (width 0) (type default))
+  )
+  (wire (pts (xy 97.79 106.68) (xy 143.51 106.68))
+    (stroke (width 0) (type default))
+  )
   (wire (pts (xy 128.27 76.2) (xy 128.27 82.55))
     (stroke (width 0) (type default))
   )
-  (wire (pts (xy 104.14 97.79) (xy 104.14 76.2))
-    (stroke (width 0) (type default))
-  )
-  (wire (pts (xy 162.56 100.33) (xy 167.64 100.33))
-    (stroke (width 0) (type default))
-  )
-  (wire (pts (xy 236.22 83.82) (xy 236.22 81.28))
-    (stroke (width 0) (type default))
-  )
-  (wire (pts (xy 104.14 76.2) (xy 128.27 76.2))
-    (stroke (width 0) (type default))
-  )
-  (wire (pts (xy 140.97 97.79) (xy 143.51 97.79))
-    (stroke (width 0) (type default))
-  )
-  (wire (pts (xy 179.07 110.49) (xy 179.07 113.03))
-    (stroke (width 0) (type default))
-  )
-  (wire (pts (xy 147.32 87.63) (xy 140.97 87.63))
-    (stroke (width 0) (type default))
-  )
-  (wire (pts (xy 179.07 113.03) (xy 179.07 120.65))
-    (stroke (width 0) (type default))
-  )
-  (wire (pts (xy 128.27 76.2) (xy 139.7 76.2))
-    (stroke (width 0) (type default))
-  )
-  (wire (pts (xy 167.64 100.33) (xy 179.07 100.33))
-    (stroke (width 0) (type default))
-  )
-  (wire (pts (xy 228.6 88.9) (xy 228.6 95.25))
-    (stroke (width 0) (type default))
-  )
-  (wire (pts (xy 228.6 118.11) (xy 228.6 105.41))
-    (stroke (width 0) (type default))
-  )
-  (wire (pts (xy 97.79 106.68) (xy 143.51 106.68))
-    (stroke (width 0) (type default))
-  )
   (wire (pts (xy 236.22 81.28) (xy 228.6 81.28))
     (stroke (width 0) (type default))
@@
   )
   (wire (pts (xy 167.64 113.03) (xy 167.64 100.33))
+    (stroke (width 0) (type default))
+  )
+  (wire (pts (xy 128.27 113.03) (xy 128.27 115.57))
     (stroke (width 0) (type default))
   )
@@
   (symbol (lib_id "Device:R_Potentiometer") (at 179.07 106.68 180) (unit 1)
     (in_bom yes) (on_board yes) (dnp no)
-    (property "Reference" "RV1(Frecuencia)" (at 180.34 105.41 0)
+    (property "Reference" "RV1(Frecuencia)1" (at 180.34 105.41 0)
       (effects (font (size 1.27 1.27)) (justify right))
     )
@@
       (project "NE555 frecuencia y pwm [Kicad]"
         (path "/cb09506a-9f8b-4169-8b76-bcea4c99a790"
-          (reference "RV1(Frecuencia)") (unit 1)
+          (reference "RV1(Frecuencia)1") (unit 1)
         )
       )
@@
     )
   )
+  (symbol (lib_id "power:PWR_FLAG") (at 128.27 113.03 270) (unit 1)
+    (in_bom yes) (on_board yes) (dnp no) (fields_autoplaced)
+    (property "Reference" "#FLG02" (at 130.175 113.03 0)
+      (effects (font (size 1.27 1.27)) hide)
+    )
+    (property "Value" "PWR_FLAG" (at 132.08 113.03 90)
+      (effects (font (size 1.27 1.27)) (justify left))
+    )
+    (property "Footprint" "" (at 128.27 113.03 0)
+      (effects (font (size 1.27 1.27)) hide)
+    )
+    (property "Datasheet" "~" (at 128.27 113.03 0)
+      (effects (font (size 1.27 1.27)) hide)
+    )
+    (pin "1")
+    (instances
+      (project "NE555 frecuencia y pwm [Kicad]"
+        (path "/cb09506a-9f8b-4169-8b76-bcea4c99a790"
+          (reference "#FLG02") (unit 1)
+        )
+      )
+    )
+  )
   (symbol (lib_id "Connector:Screw_Terminal_01x02") (at 74.93 93.98 180) (unit 1)
     (in_bom yes) (on_board yes) (dnp no)
@@
   (symbol (lib_id "Device:R_Potentiometer") (at 151.13 106.68 180) (unit 1)
     (in_bom yes) (on_board yes) (dnp no)
-    (property "Reference" "RV2(Duty)" (at 152.4 105.41 0)
+    (property "Reference" "RV2(Duty)1" (at 152.4 105.41 0)
       (effects (font (size 1.27 1.27)) (justify right))
     )
@@
       (project "NE555 frecuencia y pwm [Kicad]"
         (path "/cb09506a-9f8b-4169-8b76-bcea4c99a790"
-          (reference "RV2(Duty)") (unit 1)
-        )
-      )
+          (reference "RV2(Duty)1") (unit 1)
+        )
+      )
+    )
+  )
+  (symbol (lib_id "power:PWR_FLAG") (at 128.27 71.12 90) (unit 1)
+    (in_bom yes) (on_board yes) (dnp no) (fields_autoplaced)
+    (property "Reference" "#FLG01" (at 126.365 71.12 0)
+      (effects (font (size 1.27 1.27)) hide)
+    )
+    (property "Value" "PWR_FLAG" (at 124.46 71.12 90)
+      (effects (font (size 1.27 1.27)) (justify left))
+    )
+    (property "Footprint" "" (at 128.27 71.12 0)
+      (effects (font (size 1.27 1.27)) hide)
+    )
+    (property "Datasheet" "~" (at 128.27 71.12 0)
+      (effects (font (size 1.27 1.27)) hide)
+    )
+    (pin "1")
+    (instances
+      (project "NE555 frecuencia y pwm [Kicad]"
+        (path "/cb09506a-9f8b-4169-8b76-bcea4c99a790"
+          (reference "#FLG01") (unit 1)
+        )
+      )
