File: Circuitos/RC_square_to_sin_[Kicad]/RC_square_to_sin_[Kicad].kicad_sch (KiCad schematic)
At the start: 3 parts

Commit message: .
Parts:
- added C2, C3: 10n, symbol Device:C
- added R2, R3: 1.5k, symbol Device:R
- C1: value 10uF -> 10n
- R1: value 10k -> 1.5k
Connections:
- net 0: now also C1.1, C2.1, C3.1; no longer R1.2
- net RCline: now also C3.2, R3.2; no longer C1.2, R1.1
- net at V1.1: now also R1.1; no longer C1.1
- new net: C2.2, R2.2, R3.1
- new net: C1.2, R1.2, R2.1
Other:
- note removed: ".ic V(/RCline)=0"
